File: pcb/spinduino.brd (EAGLE design)
At the start: 78.5 x 86.8 mm, 30 parts

Commit message: add programming connector
Parts:
- added J1: (no value), ng-beacon:1X04_LOCK
- moved U$3 0.10 mm to (63.6, 41.9)
Connections:
- new net SWCLK: J1.3, U$1.4
- new net SWDIO: J1.2, U$1.5
- net GND: now also J1.4
- net V_BATT: now also J1.1
Routing:
- net SWCLK: track 0.00 -> 25.8 mm
- net GND: track 208.3 -> 232.2 mm, vias 4 -> 3
- net SWDIO: track 0.00 -> 22.3 mm
- net V_BATT: track 200.1 -> 197.4 mm
- net HALL1: track 53.6 -> 52.3 mm
Other:
- board text added: "(c) 2017, Uri Shaked"
- board text added: "Spinduino rev 1"
